Commit message: 12th October

File: src/my_r2d2/urdf/r2d2.urdf.xacro (robot description, xacro)
@@ -37,9 +37,10 @@
     <xacro:default_inertial mass="10"/>
   </link>
-  <link name="base_footprint">
-    <visual>
-      <geometry>
-        <box size="${baselen} ${width*2} 0.1+(2*${wheeldiam/2})" footprint parent
-      baselink child
+<link name="base_footprint"/>
+ <joint name="base_footprint_to_base" type="fixed">
+      <parent link="base_footprint"/>
+      <child link="base_link"/>
+      <origin xyz="0 0 ${(bodylen/2)+0.1+0.07}" />
+ </joint>
   <xacro:macro name="wheel" params="prefix suffix reflect">
     <link name="${prefix}_${suffix}_wheel">

Commit message: 6th lab

File: src/my_r2d2/urdf/r2d2.urdf.xacro (robot description, xacro)
@@ -214,4 +214,10 @@
     <xacro:default_inertial mass="1"/>
   </link>
+<link name="eye"/>
+ <joint name="box_to_eye" type="fixed">
+      <parent link="box"/>
+      <child link="eye"/>
+      <origin rpy="10 10 0" xyz="0 0 0"/>
+ </joint>
   <joint name="tobox" type="fixed">
     <parent link="head"/>

Commit message: Update r2d2.urdf.xacro

File: src/my_r2d2/urdf/r2d2.urdf.xacro (robot description, xacro)
@@ -215,9 +215,9 @@
   </link>
 <link name="eye"/>
- <joint name="box_to_eye" type="fixed">
-      <parent link="box"/>
-      <child link="eye"/>
-      <origin rpy="10 10 0" xyz="0 0 0"/>
- </joint>
+<joint name="eye_joint" type="fixed">
+    <parent link="box"/>
+    <child link="eye"/>
+    <origin xyz="-0.04 0 0" rpy="${pi/2} ${pi} ${pi/2}"/>
+  </joint>
   <joint name="tobox" type="fixed">
     <parent link="head"/>

Commit message: Start of 7th lab

File: src/my_r2d2/urdf/r2d2.urdf.xacro (robot description, xacro)
@@ -218,5 +218,5 @@
     <parent link="box"/>
     <child link="eye"/>
-    <origin xyz="-0.04 0 0" rpy="${pi/2} ${pi} ${pi/2}"/>
+    <origin xyz="0 0 0" rpy="${pi/2} ${pi} ${pi/2}"/>
   </joint>
   <joint name="tobox" type="fixed">
